Commit message: latest update
removed caps
formed meshes
no v6

File: assembly_urdf/urdf/assembly_urdf.urdf (robot description, URDF)
Before this commit: robot Assembly_URDF v6, 7 links, 6 joints
Links:
- removed link Gripper_link
- removed link Link_3
- removed link shaft_Link1
- added link gripper_link, mass 0.822220892683325; collision mesh filename=package://assembly_urdf/meshes/gripper_link.STL; visual mesh filename=package://assembly_urdf/meshes/gripper_link.STL
- added link link_3, mass 0.973698526007838; collision mesh filename=package://assembly_urdf/meshes/link_3.STL; visual mesh filename=package://assembly_urdf/meshes/link_3.STL
- added link shaft_link1, mass 0.046919956660997; collision mesh filename=package://assembly_urdf/meshes/shaft_link1.STL; visual mesh filename=package://assembly_urdf/meshes/shaft_link1.STL
- link Link_2: geometry collision mesh filename=package://assembly_urdf/meshes/Link_2.STL; visual mesh filename=package://assembly_urdf/meshes/Link_2.STL
- link base_link: mass 2.50216732502464 -> 2.50216732502463; geometry collision mesh filename=package://assembly_urdf/meshes/base_link.STL; visual mesh filename=package://assembly_urdf/meshes/base_link.STL
- link shaft_link2: mass 0.0469199566610043 -> 0.0469199566610044; geometry collision mesh filename=package://assembly_urdf/meshes/shaft_link2.STL; visual mesh filename=package://assembly_urdf/meshes/shaft_link2.STL
- link shaft_link3: mass 0.0469199566610041 -> 0.0469199566610044; geometry collision mesh filename=package://assembly_urdf/meshes/shaft_link3.STL; visual mesh filename=package://assembly_urdf/meshes/shaft_link3.STL
Joints:
- removed joint motor_1
- removed joint motor_2
- removed joint motor_3
- removed joint pitch movement
- removed joint yaw movement
- removed joint yaw_move
- added joint gripper_movement: type revolute, parent base_link, child gripper_link, origin xyz=-0.02769 0.018952 1.2402 rpy=1.5708 0 0, axis 0 0 0, limit lower=-1.5708 upper=1.5708 effort=0 velocity=0
- added joint motor_link1: type revolute, parent base_link, child shaft_link1, origin xyz=0.085 -0.067256 0.56196 rpy=1.5708 -1.5708 0, axis 0 0 0, limit lower=-1.5708 upper=1.5708 effort=0 velocity=0
- added joint motor_link2: type revolute, parent Link_2, child shaft_link2, origin xyz=0.085 -0.18 0 rpy=0 0 1.5708, axis 0 0 0, limit lower=-1.5708 upper=1.5708 effort=0 velocity=0, mimic joint=motor_link3 multiplier=1 offset=0
- added joint motor_link3: type revolute, parent link_3, child shaft_link3, origin xyz=-0.08 0 0.085 rpy=-1.5708 0 0, axis 0 0 0, limit lower=-1.5708 upper=1.5708 effort=0 velocity=0, mimic joint=motor_link2 multiplier=1 offset=0
- added joint pitch_link: type revolute, parent base_link, child Link_2, origin xyz=0.00028402 -0.060596 0.71296 rpy=-1.5708 0 -1.5708, axis 0 0 0, limit lower=-1.5708 upper=1.5708 effort=0 velocity=0
- added joint yaw_link: type revolute, parent base_link, child link_3, origin xyz=-0.0013889 -0.060856 0.96396 rpy=0.2264 1.5708 -1.3444, axis 0 0 0, limit lower=-1.5708 upper=1.5708 effort=0 velocity=0
